File: zasilacz.sch (EAGLE design)
At the start: 22 parts, among them Q1 STH60N10FI, Q2 FDN360P, Q3 FDN360P, Q4 STH60N10FI, Q5 FDN360P, Q7 STH60N10FI, X1 Motor_A, X2 Motor_A

Commit message: Add files via upload
Parts:
- removed L5: (no value), ngspice-simulation:L
- removed SMT32F0_DISCOVERY1: STM32F0_DISCOVERY, stm32f0discovery:STM32F0_DISCOVERY
- removed X1, X2: Motor_A, con-phoenix-3501:1751248
- added C10, C11, C12, C13, C14, C2, C3, C7, C8, C9: (no value), rcl:C-EU025-024X044
- added D1: 1N4004, diode:1N4004
- added DISP_CATHODE: 87758-1616, con-molex:87758-1616
- added F1: (no value), fuse:SH25
- added FAN_CONNECTOR, OUTPUT_CONNECTOR, PWR_SWITCH: 22-23-2021, con-molex:22-23-2021
- added I_DISP_ANODE1, V_DISP_ANODE: 22-23-2031, con-molex:22-23-2031
- added I_ENC, V_ENC: 22-23-2051, con-molex:22-23-2051
- added L2, L3: (no value), rcl:L-EU0207/10
- added Q10, Q11, Q12, Q13, Q9: 2N4126, transistor-pnp:2N4126
- added Q6, Q8: IRF4905, transistor-power:IRF4905
- added R10, R11, R12, R13, R14, R15, R16, R17, R18, R19, R2, R20, R21, R3, R4, R7, R8, R9, R_SENSE: (no value), rcl:R-EU_0309/10
- added U1: STM32L100C-DISCO, STM32L100C-DISCO:STM32L100C-DISCO
- C4, C5, C6: device ngspice-simulation:C -> rcl:C-EU025-024X044
- IC1: value (none) -> 7805TV; device linear-technology:LT1129CST5 -> linear:7805TV
- L1, L4: device ngspice-simulation:L -> rcl:L-EU0207/10
- Q2: value FDN360P -> IRF4905; device transistor-power:FDN360P -> transistor-power:IRF4905
- Q3, Q5: value FDN360P -> STH60N10FI; device transistor-power:FDN360P -> transistor-power:STH60N10FI
- Q4: value STH60N10FI -> IRF4905; device transistor-power:STH60N10FI -> transistor-power:IRF4905
- Q7: value STH60N10FI -> 2N4126; device transistor-power:STH60N10FI -> transistor-pnp:2N4126
- R1, R5, R6: device ngspice-simulation:R -> rcl:R-EU_0309/10
Connections:
- new net 0VAC: TR1.P2
- new net 230VAC: PWR_SWITCH-2.S
- new net 3V3: I_ENC-4.S, U1.3V, V_ENC-4.S
- new net 5V: C14.1, IC1.VO, Q10.C, Q11.C, Q12.C, Q13.C, Q7.C, Q9.C, U1.5V
- new net FAN_PWM: R8.2
- new net N$13: C7.2
- new net N$14: R9.2, U1.PB14
- new net N$19: C10.1, Q6.G, R6.1
- new net N$20: C9.2
- new net N$21: Q10.E, V_DISP_ANODE-3.S
- new net N$22: C10.2
- new net N$23: F1.2, TR1.P1
- new net N$24: Q7.B, R10.1
- new net N$25: Q6.D
- new net N$26: Q9.B, R9.1
- new net N$29: D1.C, L4.1, Q8.S
- new net N$30: Q10.B, R7.1
- new net N$31: C13.1, Q8.G, R8.1
- new net N$32: Q9.E, V_DISP_ANODE-2.S
- new net N$33: C13.2
- new net N$34: C11.2, D1.A, FAN_CONNECTOR-2.S
- new net N$35: Q8.D
- new net N$36: C11.1, FAN_CONNECTOR-1.S, L4.2
- new net N$37: Q7.E, V_DISP_ANODE-1.S
- new net N$38: R11.2, U1.PC6
- new net N$39: R12.2, U1.PC7
- new net N$40: R13.2, U1.PC8
- new net N$41: Q11.B, R13.1
- new net N$42: I_DISP_ANODE1-3.S, Q13.E
- new net N$43: I_DISP_ANODE1-2.S, Q12.E
- new net N$44: I_DISP_ANODE1-1.S, Q11.E
- new net N$45: Q12.B, R12.1
- new net N$46: Q13.B, R11.1
- new net N$47: DISP_CATHODE-1.S, DISP_CATHODE-2.S, R14.2
- new net N$48: DISP_CATHODE-3.S, DISP_CATHODE-4.S, R15.2
- new net N$49: DISP_CATHODE-5.S, DISP_CATHODE-6.S, R16.2
- new net N$50: DISP_CATHODE-7.S, DISP_CATHODE-8.S, R17.2
- new net N$51: DISP_CATHODE-10.S, DISP_CATHODE-9.S, R18.2
- new net N$52: DISP_CATHODE-11.S, DISP_CATHODE-12.S, R19.2
- new net N$53: DISP_CATHODE-13.S, DISP_CATHODE-14.S, R20.2
- new net N$54: DISP_CATHODE-15.S, DISP_CATHODE-16.S, R21.2
- new net N$55: R21.1, U1.PC11
- new net N$56: R14.1, U1.PB7
- new net N$57: R15.1, U1.PB6
- new net N$58: R16.1, U1.PB5
- new net N$59: R17.1, U1.PB4
- new net N$60: R18.1, U1.PB3
- new net N$61: R19.1, U1.PD2
- new net N$62: R20.1, U1.PC12
- new net N$63: I_ENC-1.S, U1.PB12
- new net N$64: I_ENC-2.S, U1.PB11
- new net N$65: I_ENC-3.S, U1.PB10
- new net N$66: U1.PB2, V_ENC-1.S
- new net N$67: U1.PB1, V_ENC-2.S
- new net N$68: U1.PB0, V_ENC-3.S
- new net N$69: F1.1, PWR_SWITCH-1.S
- new net PH1N: R1.1
- new net PH1P: R2.2
- new net PH2N: R3.1
- new net PH2P: R4.2
- new net PH3N: R5.1
- new net PH3OUT+: C2.1, C5.1, C8.1, L1.2, L2.2, L3.2, R_SENSE.1
- new net PH3OUT-: C2.2, C5.2, C8.2, OUTPUT_CONNECTOR-2.S, Q1.S, Q3.S, Q5.S
- new net PH3P: R6.2
- net GND: now also B1.AC2, C1.2, C12.2, C14.2, IC1.GND, I_ENC-5.S, U1.P2_GND2, V_ENC-5.S; no longer IC1G$1.GND, SMT32F0_DISCOVERY1.GND5, TR1.P2
- net N$1: now also L2.1, Q3.D, Q4.S; no longer L1.1, R1.2
- net N$10: now also C4.2; no longer Q4.D, Q5.D, R6.1
- net N$11: now also C4.1, Q2.G, R2.1; no longer C1.1, C5.1, C6.1, L1.2, L4.2, L5.2, X1-1.K
- net N$12: now also Q2.D; no longer Q7.G, SMT32F0_DISCOVERY1.PA0
- net N$15: now also Q4.D; no longer B1.AC1, C4.1, IC1G$1.IN, Q2.S, Q3.S, Q5.S
- net N$16: now also R10.2, U1.PB15; no longer Q3.G, SMT32F0_DISCOVERY1.PC3
- net N$17: now also L3.1, Q5.D, Q6.S; no longer Q5.G, SMT32F0_DISCOVERY1.PC1
- net N$18: now also C9.1, Q5.G, R5.2; no longer Q4.G, SMT32F0_DISCOVERY1.PC0
- net N$2: now also OUTPUT_CONNECTOR-1.S, R_SENSE.2; no longer IC1G$1.OUT, SMT32F0_DISCOVERY1.5V
- net N$3: now also C6.1, Q3.G, R3.2; no longer Q2.D, Q7.D, R1.1
- net N$4: now also C7.1, Q4.G, R4.1; no longer Q1.G, SMT32F0_DISCOVERY1.PC2
- net N$5: now also R7.2, U1.PB13; no longer L4.1, R5.2
- net N$6: now also L1.1, Q2.S; no longer Q3.D, R5.1
- net N$7: now also C6.2; no longer Q2.G, SMT32F0_DISCOVERY1.PA1
- net N$8: now also C3.1, Q1.G, R1.2; no longer B1.AC2, C1.2, C4.2, C5.2, C6.2, Q1.S, Q4.S, Q7.S, X2-1.K
- net N$9: now also C3.2; no longer L5.1, R6.2
- net VCC: now also B1.AC1, C1.1, C12.1, IC1.VI; no longer TR1.P1
Other:
- moved on the sheet: B1, C1, C4, C5, C6, Q1, Q3, Q5, R1, R5, R6, TR1

Commit message: Add files via upload
Parts:
- removed B1: (no value), rectifier:B-DIL
- removed F1: (no value), fuse:SH25
- removed PWR_SWITCH: 22-23-2021, con-molex:22-23-2021
- removed TR1: (no value), trafo:EI30-1
- added B2: (no value), rectifier:GBU4
- added TRAFO: 22-23-2021, con-molex:22-23-2021
- Q1, Q3, Q5: value STH60N10FI -> (none); device transistor-power:STH60N10FI -> transistor-power:PMOSFET_NTO220BV
- Q2, Q4, Q6, Q8: value IRF4905 -> (none); device transistor-power:IRF4905 -> transistor-power:PMOSFET_PTO220BV
Connections:
- removed net 0VAC: TR1.P2
- removed net 230VAC: PWR_SWITCH-2.S
- removed net N$28 (its old number): B1.+, TR1.S3
- removed net N$55 (its old number): R21.1, U1.PC11
- removed net N$56 (its old number): R14.1, U1.PB7
- removed net N$57 (its old number): R15.1, U1.PB6
- removed net N$58 (its old number): R16.1, U1.PB5
- removed net N$59 (its old number): R17.1, U1.PB4
- removed net N$69: F1.1, PWR_SWITCH-1.S
- new net N$63: R12.2, U1.PC4
- new net N$64: R11.2, U1.PA7
- new net N$65: R10.2, U1.PA6
- new net N$66: R9.2, U1.PA5
- new net N$67: R7.2, U1.PA4
- net GND: now also B2.-; no longer B1.AC2
- net N$14: now also R20.1, U1.PC14; no longer R9.2, U1.PB14
- net N$16: now also R19.1, U1.PC15; no longer R10.2, U1.PB15
- net N$23: now also B2.AC2, TRAFO-2.S; no longer F1.2, TR1.P1
- net N$27: now also B2.AC1, TRAFO-1.S; no longer B1.-, TR1.S4
- net N$38: now also R18.1, U1.PH0; no longer R11.2, U1.PC6
- net N$39: now also R17.1, U1.PH1; no longer R12.2, U1.PC7
- net N$40: now also R16.1, U1.P1_GND1; no longer R13.2, U1.PC8
- net N$5: now also R21.1, U1.PC13; no longer R7.2, U1.PB13
- net N$60: now also R15.1, U1.NRST; no longer R18.1, U1.PB3
- net N$61: now also R14.1, U1.PC0; no longer R19.1, U1.PD2
- net N$62: now also R13.2, U1.PC5; no longer R20.1, U1.PC12
- net VCC: now also B2.+; no longer B1.AC1
Other:
- moved on the sheet: C1, C10, C11, C12, C13, C14, C4, C7, D1, DISP_CATHODE-1, DISP_CATHODE-10, DISP_CATHODE-11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

Commit message: Add files via upload
Parts:
- removed C13: (no value), rcl:C-EU025-024X044
- added D2, D3, D4: (no value), diode:SCHOTTKY-DIODEDO35-7
- added U2, U3, U4: IR2101, IR2101:IR2101
- Q2, Q4, Q6: device transistor-power:PMOSFET_PTO220BV -> transistor-power:PMOSFET_NTO220BV
Connections:
- removed net N$1: L2.1, Q3.D, Q4.S
- removed net N$10: C4.2
- removed net N$12: Q2.D
- removed net N$13: C7.2
- removed net N$15: Q4.D
- removed net N$17: L3.1, Q5.D, Q6.S
- removed net N$20: C9.2
- removed net N$22: C10.2
- removed net N$25: Q6.D
- removed net N$33: C13.2
- removed net N$35: Q8.D
- removed net N$6: L1.1, Q1.D, Q2.S
- removed net N$7: C6.2
- removed net N$9: C3.2
- new net PH1VS: C3.2, L1.1, Q1.D, Q6.D, U2.VS
- new net PH1_HIN: U1.PA13, U2.HIN
- new net PH1_LIN: U1.PA12, U2.LIN
- new net PH2VS: C6.2, L2.1, Q3.D, Q4.D, U3.VS
- new net PH2_HIN: U1.PA11, U3.HIN
- new net PH2_LIN: U1.PA10, U3.LIN
- new net PH3VS: C9.2, L3.1, Q2.D, Q5.D, U4.VS
- new net PH3_HIN: U1.PA9, U4.HIN
- new net PH3_LIN: U1.PA8, U4.LIN
- new net VB: C3.1, C6.1, C9.1, D2.C, D3.C, D4.C, U2.VB, U3.VB, U4.VB
- net 3V3: now also C10.1, C4.1, C7.1, D2.A, D3.A, D4.A, Q10.E, Q11.E, Q12.E, Q13.E, Q7.E, Q9.E, U2.VCC, U3.VCC, U4.VCC
- net 5V: no longer Q10.C, Q11.C, Q12.C, Q13.C, Q7.C, Q9.C
- net GND: now also C10.2, C4.2, C7.2, U2.COM, U3.COM, U4.COM
- net N$11: now also Q6.G; no longer C4.1, Q2.G
- net N$18: no longer C9.1
- net N$19: now also Q2.G; no longer C10.1, Q6.G
- net N$21: now also Q13.C; no longer Q10.E
- net N$24: now also Q10.B; no longer Q7.B
- net N$26: now also Q12.B; no longer Q9.B
- net N$29: now also Q8.D; no longer Q8.S
- net N$3: no longer C6.1
- net N$30: now also Q13.B; no longer Q10.B
- net N$31: no longer C13.1
- net N$32: now also Q12.C; no longer Q9.E
- net N$37: now also Q10.C; no longer Q7.E
- net N$4: no longer C7.1
- net N$42: now also Q9.C; no longer Q13.E
- net N$43: now also Q7.C; no longer Q12.E
- net N$44: now also Q11.C; no longer Q11.E
- net N$45: now also Q7.B; no longer Q12.B
- net N$46: now also Q9.B; no longer Q13.B
- net N$8: no longer C3.1
- net PH1N: now also U2.LO
- net PH1P: now also U2.HO
- net PH2N: now also U3.LO
- net PH2P: now also U3.HO
- net PH3N: now also U4.LO
- net PH3P: now also U4.HO
- net VCC: now also Q2.S, Q4.S, Q6.S, Q8.S
Other:
- moved on the sheet: C10, C3, C4, C6, C7, C9, Q10, Q11, Q12, Q13, Q7, Q9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
