File: Projekt EAGLE/zasilacz.sch (EAGLE design)
At the start: 70 parts, among them IC1 7805TV, Q10 2N4126, Q11 2N4126, Q12 2N4126, Q13 2N4126, Q7 2N4126, Q9 2N4126, U1 STM32L100C-DISCO, U2 IR2101, U3 IR2101, U4 IR2101

Commit message: .
Parts:
- added C13: (no value), rcl:C-EU025-024X044
- added D10, D7, D8, D9: (no value), diode:ZENER-DIODEDO34-7
- added IC3: 7812TV, linear:7812TV
- added L5: (no value), rcl:L-EU0207/10
- added R22, R23, R24, R25, R26: (no value), rcl:R-EU_0309/10
- added T1: 2SC1815, transistor:2SC1815
- added U$1: AD8410AD8410_V1, AD8410:AD8410AD8410_V1
Connections:
- net N$2 renamed -R_SENSE
- removed net N$31: Q8.G, R8.1
- removed net N$34: C11.2, D1.A, FAN_CONNECTOR-2.S
- removed net N$36: C11.1, FAN_CONNECTOR-1.S, L4.2
- removed net PH3OUT+: C2.1, C5.1, C8.1, L1.2, L2.2, L3.2, R_SENSE.1
- removed net PH3OUT-: C2.2, C5.2, C8.2, OUTPUT_CONNECTOR-2.S, Q1.S, Q3.S, Q5.S
- new net +R_SENSE: C2.1, C5.1, C8.1, L1.2, L2.2, L3.2, R24.1, R_SENSE.1
- new net I_MEASURE_OUT: U$1.OUT
- new net N$1: Q8.G, R8.2, T1.C
- new net N$10: U1.PB15
- new net N$12: U1.PB14
- new net N$13: U1.PB13
- new net N$15: D7.C
- new net N$2: R26.2, T1.B
- new net N$6: B2.+, L5.1
- new net N$7: C13.1, IC3.VI
- new net N$9: U$1.VREF_1, U$1.VS
- new net UWY: C11.1, FAN_CONNECTOR-1.S, L4.2, R22.1
- new net V_MEASURE_FAN: D10.C, D7.A, R22.2, R23.1
- new net V_MEASURE_OUT: D8.A, D9.C, R24.2, R25.1
- net 3V3: now also D8.C
- net FAN_PWM: now also R26.1; no longer R8.2
- net GND: now also C11.2, C13.2, C2.2, C5.2, C8.2, D1.A, D10.A, D9.A, FAN_CONNECTOR-2.S, IC3.GND, OUTPUT_CONNECTOR-2.S, Q1.S, Q3.S, Q5.S, R23.2, R25.2, T1.E, U$1.GND, U$1.VREF_2
- net VCC: now also IC3.VO, L5.2, R8.1; no longer B2.+
Other:
- moved on the sheet: B2, C1, C10, C11, C12, C14, C3, C4, C6, C7, C9, D1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

Commit message: .
Connections:
- removed net N$7: C13.1, IC3.VI
- net VCC: now also C13.1, IC3.VI
Changed lines of the file:
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@@
 <junction x="246.38" y="-144.78"/>
+</segment>
+<segment>
+<pinref part="C13" gate="G$1" pin="1"/>
+<wire x1="358.14" y1="78.74" x2="358.14" y2="83.82" width="0.1524" layer="91"/>
+<wire x1="358.14" y1="83.82" x2="360.68" y2="83.82" width="0.1524" layer="91"/>
+<label x="355.6" y="83.82" size="1.778" layer="95" rot="MR0" xref="yes"/>
+<wire x1="358.14" y1="83.82" x2="355.6" y2="83.82" width="0.1524" layer="91"/>
+<junction x="358.14" y="83.82"/>
+<pinref part="IC3" gate="A1" pin="VI"/>
 </segment>
 </net>
@@
 </segment>
 </net>
-<net name="N$7" class="0">
-<segment>
-<pinref part="C13" gate="G$1" pin="1"/>
-<wire x1="358.14" y1="78.74" x2="358.14" y2="83.82" width="0.1524" layer="91"/>
-<wire x1="358.14" y1="83.82" x2="360.68" y2="83.82" width="0.1524" layer="91"/>
-<label x="355.6" y="83.82" size="1.778" layer="95" rot="MR0" xref="yes"/>
-<wire x1="358.14" y1="83.82" x2="355.6" y2="83.82" width="0.1524" layer="91"/>
-<junction x="358.14" y="83.82"/>
-<pinref part="IC3" gate="A1" pin="VI"/>
-</segment>
-</net>

Commit message: Add files via upload
Parts:
- removed DISP_CATHODE: 87758-1616, con-molex:87758-1616
- added C15, C16, C17, C18, C19, C22: (no value), rcl:C-EU025-024X044
- added X1, X2: 22-23-2081, con-molex:22-23-2081
- C1: device ngspice-simulation:C -> rcl:C-EU025-024X044
Connections:
- removed net N$12: U1.PB14
- removed net N$13: U1.PB13
- removed net N$15: D7.C
- removed net N$38: R18.1, U1.PH0
- removed net N$39: R17.1, U1.PH1
- removed net N$40: R16.1, U1.P1_GND1
- removed net N$60: R15.1, U1.NRST
- removed net N$61: R14.1, U1.PC0
- new net N$17: R18.1, U1.PC3
- new net N$20: R19.1, U1.PC2
- new net N$22: R20.1, U1.PC1
- new net N$25: R21.1, U1.PC0
- new net N$7: R15.1, U1.PA2
- net +R_SENSE: now also U$1.+IN; no longer R24.1
- net -R_SENSE: now also R24.1, U$1.-IN
- net 3V3: now also C17.1, C18.1, C19.1, D7.C
- net 5V: now also U1.P1_VDD, U1.P2_VDD, U1.P2_VDD1
- net FAN_PWM: now also U1.PB13
- net GND: now also C1.1, C15.1, C16.1, C17.2, C18.2, C19.2, C22.1, U1.P1_GND, U1.P1_GND1, U1.P1_GND2, U1.P1_GND3, U1.P2_GND, U1.P2_GND1; no longer C1.2
- net I_MEASURE_OUT: now also U1.PB15
- net N$10: now also C12.1, IC1.VI, IC3.VO; no longer U1.PB15
- net N$14: now also R16.1, U1.PA1; no longer R20.1, U1.PC14
- net N$16: now also R17.1, U1.PA0; no longer R19.1, U1.PC15
- net N$47: now also X1-1.S, X2-1.S; no longer DISP_CATHODE-1.S, DISP_CATHODE-2.S
- net N$48: now also X1-2.S, X2-2.S; no longer DISP_CATHODE-3.S, DISP_CATHODE-4.S
- net N$49: now also X1-3.S, X2-3.S; no longer DISP_CATHODE-5.S, DISP_CATHODE-6.S
- net N$5: now also R14.1, U1.PA3; no longer R21.1, U1.PC13
- net N$50: now also X1-4.S, X2-4.S; no longer DISP_CATHODE-7.S, DISP_CATHODE-8.S
- net N$51: now also X1-5.S, X2-5.S; no longer DISP_CATHODE-10.S, DISP_CATHODE-9.S
- net N$52: now also X1-6.S, X2-6.S; no longer DISP_CATHODE-11.S, DISP_CATHODE-12.S
- net N$53: now also X1-7.S, X2-7.S; no longer DISP_CATHODE-13.S, DISP_CATHODE-14.S
- net N$54: now also X1-8.S, X2-8.S; no longer DISP_CATHODE-15.S, DISP_CATHODE-16.S
- net N$9: now also C22.2
- net VCC: now also C1.2, C15.2, C16.2; no longer C1.1, C12.1, IC1.VI, IC3.VO
- net V_MEASURE_FAN: now also U1.PB14
- net V_MEASURE_OUT: now also U1.PC6
Other:
- moved on the sheet: C1, C10, C4, C7, R14, R15, R16, R17, R18, R19, R20, R21

Commit message: Add files via upload
Parts:
- removed B2: (no value), rectifier:GBU4
- removed C3, C6, C9: (no value), rcl:C-EU025-024X044
- removed D4: (no value), diode:SCHOTTKY-DIODEDO35-7
- removed L1, L2, L3, L4, L5: (no value), rcl:L-EU0207/10
- removed R8, R_SENSE: (no value), rcl:R-EU_0309/10
- added B9: RECTIFIER-2KBP, rectifier:RECTIFIER-2KBP
- added C20, C21: (no value), rcl:C-EUC0603K
- added D5: SB120, diode:SB120
- added R27: (no value), rcl:R-EU_R2512
- added R28: (no value), rcl:R-EU_0207/10
- added U$2, U$3, U$4, U$5: 5256-RC5256-RC, rcl:5256-RC5256-RC
- added U$6: C_MOJE_GRID12MM5, rcl:C_MOJE_GRID12MM5
- C1, C2, C5, C8: device rcl:C-EU025-024X044 -> rcl:CPOL-EUE5-13
- C11: device rcl:C-EU025-024X044 -> rcl:C-EUC0603K
- D2, D3: value (none) -> SB120; device diode:SCHOTTKY-DIODEDO35-7 -> diode:SB120
- R22, R24: device rcl:R-EU_0309/10 -> rcl:R-EU_0207/12
Connections:
- removed net N$6: B2.+, L5.1
- net +R_SENSE: now also C1.+, C2.+, C5.+, R27.1, U$2.2, U$3.2, U$4.2; no longer C2.1, C5.1, C8.1, L1.2, L2.2, L3.2, R_SENSE.1
- net -R_SENSE: now also R22.2, R27.2; no longer R24.1, R_SENSE.2
- net 3V3: now also D5.A; no longer D4.A
- net FAN_PWM: now also U1.PB9; no longer U1.PB13
- net GND: now also B9.AC2, C1.-, C2.-, C5.-, C8.-, U$6.2; no longer B2.-, C1.1, C11.2, C2.2, C5.2, C8.2
- net N$1: now also R28.2; no longer R8.2
- net N$23: now also B9.+; no longer B2.AC2
- net N$27: now also B9.-; no longer B2.AC1
- net N$29: now also U$5.1; no longer L4.1
- net PH1VS: now also C11.2, U$3.1; no longer C3.2, L1.1
- net PH1_HIN: now also U1.PB7; no longer U1.PA13
- net PH1_LIN: now also U1.PB6; no longer U1.PA12
- net PH2VS: now also C20.2, U$2.1; no longer C6.2, L2.1
- net PH3VS: now also C21.2, U$4.1; no longer C9.2, L3.1
- net UWY: now also C8.+, R24.2, U$5.2; no longer C11.1, L4.2, R22.1
- net VB: now also C11.1, C20.1, C21.1, D5.C; no longer C3.1, C6.1, C9.1, D4.C
- net VCC: now also B9.AC1, R28.1, U$6.1; no longer C1.2, L5.2, R8.1
- net V_MEASURE_FAN: now also R24.1; no longer R22.2
- net V_MEASURE_OUT: now also R22.1; no longer R24.2
Other:
- moved on the sheet: C11, R22, R24

Commit message: Add files via upload
Connections:
- net PH1VS: now also Q6.S; no longer Q6.D
- net PH2VS: now also Q4.S; no longer Q4.D
- net PH3VS: now also Q2.S; no longer Q2.D
- net VCC: now also Q2.D, Q4.D, Q6.D; no longer Q2.S, Q4.S, Q6.S
